Commit message: more work

File: urdf/bullet.urdf (robot description, URDF)
Before this commit: robot bullet, 3 links, 2 joints
Links:
- added link base_footprint
- added link scan_link; visual cylinder length=0.07 radius=0.03
Joints:
- added joint footprint_joint: type fixed, parent base_link, child base_footprint, origin xyz=0 0 -0.06 rpy=0 0 0
- added joint scan_joint: type fixed, parent scan_link, child base_link
