Commit message: work in progress

File: sodacan/urdf/platform3.urdf (robot description, URDF)
Before this commit: robot platform, 7 links, 6 joints
Joints:
- removed joint base_link_to_camera_link
- added joint Footprint_to_camera_link: type fixed, parent base_footprint, child camera_link, origin xyz=0.08 0 0.1 rpy=${-pi/2} 0 ${-pi/2}

Commit message: work in progress

File: sodacan/urdf/platform3.urdf (robot description, URDF)
Before this commit: robot platform, 7 links, 6 joints
Joints:
- joint Footprint_to_camera_link: origin xyz=0.08 0 0.1 rpy=${-pi/2} 0 ${-pi/2} -> xyz=0.08 0 0.1 rpy=${-pi/2 - 0.3} 0 ${-pi/2}
